File: projekt1.kicad_sch (KiCad schematic)
At the start: 71 parts, among them IC1 TPS563300DRLR, J1 V1, J2 V1, J4 PN532 connector, K1 1461103-1, K2 SANYOU_SRD_Form_B, Q1 MMBT3904, Q2 MMBT3904, SW1 SW_Push, SW10 SW_Push, SW11 SW_Push, SW12 SW_Push, SW2 SW_Push, SW3 SW_Push, SW4 SW_Push, SW5 SW_Push, SW6 SW_Push, SW7 SW_Push, SW8 SW_Push, SW9 SW_Push, U1 STM32F030C8Tx, U2 ESP-12E, U4 LTV-824, Y1 ABM3-8.000MHZ-D2Y

Commit message: rfid module
Parts:
- removed J4: PN532 connector, Connector_PinHeader_1.00mm:PinHeader_1x04_P1.00mm_Vertical, symbol Connector:Conn_01x04_Pin
- added P1: RFID-RC522-MODULE, RF_Module:ESP-07, symbol rfid-rc522-module:RFID-RC522-MODULE
Connections:
- net GND: now also P1.6 (GND)
- net I2C1_SCL: now also P1.2 (SCL)
- net I2C1_SDA: now also P1.1 (SDA)
- net VDD: now also P1.8 (3.3V)
- no-connect marks 40 -> 44
Changed lines of the file:
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@@
   (no_connect (at 55.88 90.17))
   (no_connect (at 160.02 50.8))
+  (no_connect (at 187.96 114.3))
   (no_connect (at 55.88 54.61))
   (no_connect (at 160.02 63.5))
@@
   (no_connect (at 55.88 52.07))
   (no_connect (at 92.71 138.43))
+  (no_connect (at 187.96 102.87))
+  (no_connect (at 187.96 118.11))
   (no_connect (at 86.36 67.31))
   (no_connect (at 55.88 69.85))
@@
   (no_connect (at 55.88 77.47))
   (no_connect (at 129.54 66.04))
+  (no_connect (at 187.96 110.49))
   (no_connect (at 129.54 63.5))
   (no_connect (at 160.02 53.34))
@@
     (stroke (width 0) (type default))
   )
-  (wire (pts (xy 207.01 119.38) (xy 213.36 119.38))
-    (stroke (width 0) (type default))
-  )
   (wire (pts (xy 242.57 17.78) (xy 255.27 17.78))
     (stroke (width 0) (type default))
@@
     (stroke (width 0) (type default))
   )
-  (wire (pts (xy 207.01 116.84) (xy 213.36 116.84))
-    (stroke (width 0) (type default))
-  )
   (wire (pts (xy 204.47 64.77) (xy 205.74 64.77))
     (stroke (width 0) (type default))
@@
     (stroke (width 0) (type default))
   )
+  (wire (pts (xy 193.04 106.68) (xy 187.96 106.68))
+    (stroke (width 0) (type default))
+  )
   (wire (pts (xy 33.02 181.61) (xy 33.02 177.8))
     (stroke (width 0) (type default))
@@
     (stroke (width 0) (type dash))
   )
-  (wire (pts (xy 207.01 111.76) (xy 213.36 111.76))
-    (stroke (width 0) (type default))
-  )
   (wire (pts (xy 36.83 25.4) (xy 48.26 25.4))
     (stroke (width 0) (type default))
@@
   )
   (wire (pts (xy 43.18 172.72) (xy 45.72 172.72))
-    (stroke (width 0) (type default))
-  )
-  (wire (pts (xy 207.01 114.3) (xy 213.36 114.3))
     (stroke (width 0) (type default))
   )
@@
     (effects (font (size 1.27 1.27)) (justify right bottom))
   )
-  (label "I2C1_SCL" (at 213.36 116.84 0) (fields_autoplaced)
-    (effects (font (size 1.27 1.27)) (justify left bottom))
-  )
   (label "V2_Close" (at 87.63 39.37 0) (fields_autoplaced)
     (effects (font (size 1.27 1.27)) (justify left bottom))
   )
+  (label "VDD" (at 187.96 99.06 0) (fields_autoplaced)
+    (effects (font (size 1.27 1.27)) (justify left bottom))
+  )
   (label "ROW1" (at 19.05 144.78 180) (fields_autoplaced)
     (effects (font (size 1.27 1.27)) (justify right bottom))
@@
     (effects (font (size 1.27 1.27)) (justify right bottom))
   )
+  (label "I2C1_SCL" (at 187.96 121.92 0) (fields_autoplaced)
+    (effects (font (size 1.27 1.27)) (justify left bottom))
+  )
   (label "ROW3" (at 19.05 177.8 180) (fields_autoplaced)
     (effects (font (size 1.27 1.27)) (justify right bottom))
   )
+  (label "I2C1_SDA" (at 187.96 125.73 0) (fields_autoplaced)
+    (effects (font (size 1.27 1.27)) (justify left bottom))
+  )
   (label "Relay2_NC" (at 118.11 95.25 180) (fields_autoplaced)
     (effects (font (size 1.27 1.27)) (justify right bottom))
@@
   (label "+24V" (at 118.11 105.41 180) (fields_autoplaced)
     (effects (font (size 1.27 1.27)) (justify right bottom))
-  )
-  (label "I2C1_SDA" (at 213.36 114.3 0) (fields_autoplaced)
-    (effects (font (size 1.27 1.27)) (justify left bottom))
   )
   (label "COL1" (at 45.72 190.5 270) (fields_autoplaced)
@@
     )
   )
-  (symbol (lib_id "power:GND") (at 213.36 119.38 0) (unit 1)
-    (in_bom yes) (on_board yes) (dnp no)
-    (property "Reference" "#PWR018" (at 213.36 125.73 0)
-      (effects (font (size 1.27 1.27)) hide)
-    )
-    (property "Value" "GND" (at 213.36 123.825 0)
-      (effects (font (size 1.27 1.27)))
-    )
-    (property "Footprint" "" (at 213.36 119.38 0)
-      (effects (font (size 1.27 1.27)) hide)
-    )
-    (property "Datasheet" "" (at 213.36 119.38 0)
-      (effects (font (size 1.27 1.27)) hide)
-    )
-    (pin "1")
-    (instances
-      (project "projekt1"
-        (path "/5c680b0f-7f46-4261-a30f-11ae0254e690"
-          (reference "#PWR018") (unit 1)
-        )
-      )
-    )
-  )
   (symbol (lib_id "Device:C") (at 107.95 170.18 90) (unit 1)
     (in_bom yes) (on_board yes) (dnp no)
@@
         (path "/e73816df-ff4c-47c2-ad95-54701b1a57bc"
           (reference "C?") (unit 1)
+        )
+      )
+    )
+  )
+  (symbol (lib_id "rfid-rc522-module:RFID-RC522-MODULE") (at 173.99 111.76 90) (unit 1)
+    (in_bom yes) (on_board yes) (dnp no) (fields_autoplaced)
+    (property "Reference" "P1" (at 173.355 88.9 90)
+      (effects (font (size 1.524 1.524)))
+    )
+    (property "Value" "RFID-RC522-MODULE" (at 173.355 91.44 90)
+      (effects (font (size 1.524 1.524)))
+    )
+    (property "Footprint" "RF_Module:ESP-07" (at 173.355 93.98 90)
+      (effects (font (size 1.524 1.524)))
+    )
+    (property "Datasheet" "" (at 173.99 111.76 0)
+      (effects (font (size 1.524 1.524)))
+    )
+    (pin "1")
+    (pin "2")
+    (pin "3")
+    (pin "4")
+    (pin "5")
+    (pin "6")
+    (pin "7")
+    (pin "8")
+    (instances
+      (project "projekt1"
+        (path "/5c680b0f-7f46-4261-a30f-11ae0254e690"
+          (reference "P1") (unit 1)
+        )
+      )
+      (project "access-control"
+        (path "/6e11f43c-51f2-4c65-8bff-1c594433a76d"
+          (reference "P1") (unit 1)
         )
       )
@@
     )
   )
+  (symbol (lib_id "power:GND") (at 193.04 106.68 0) (unit 1)
+    (in_bom yes) (on_board yes) (dnp no)
+    (property "Reference" "#PWR018" (at 193.04 113.03 0)
+      (effects (font (size 1.27 1.27)) hide)
+    )
+    (property "Value" "GND" (at 193.04 111.125 0)
+      (effects (font (size 1.27 1.27)))
+    )
+    (property "Footprint" "" (at 193.04 106.68 0)
+      (effects (font (size 1.27 1.27)) hide)
+    )
+    (property "Datasheet" "" (at 193.04 106.68 0)
+      (effects (font (size 1.27 1.27)) hide)
+    )
+    (pin "1")
+    (instances
+      (project "projekt1"
+        (path "/5c680b0f-7f46-4261-a30f-11ae0254e690"
+          (reference "#PWR018") (unit 1)
+        )
+      )
+    )
+  )
   (symbol (lib_id "Device:L") (at 127 134.62 0) (unit 1)
     (in_bom yes) (on_board yes) (dnp no)
@@
         (path "/5c680b0f-7f46-4261-a30f-11ae0254e690"
           (reference "#PWR02") (unit 1)
-        )
-      )
-    )
-  )
-  (symbol (lib_id "power:VDD") (at 213.36 111.76 0) (unit 1)
-    (in_bom yes) (on_board yes) (dnp no) (fields_autoplaced)
-    (property "Reference" "#PWR019" (at 213.36 115.57 0)
-      (effects (font (size 1.27 1.27)) hide)
-    )
-    (property "Value" "VDD" (at 213.36 106.68 0)
-      (effects (font (size 1.27 1.27)))
-    )
-    (property "Footprint" "" (at 213.36 111.76 0)
-      (effects (font (size 1.27 1.27)) hide)
-    )
-    (property "Datasheet" "" (at 213.36 111.76 0)
-      (effects (font (size 1.27 1.27)) hide)
-    )
-    (pin "1")
-    (instances
-      (project "projekt1"
-        (path "/5c680b0f-7f46-4261-a30f-11ae0254e690"
-          (reference "#PWR019") (unit 1)
         )
       )
@@
         )
       )
-    )
-  )
-  (symbol (lib_id "Connector:Conn_01x04_Pin") (at 201.93 114.3 0) (unit 1)
-    (in_bom yes) (on_board yes) (dnp no) (fields_autoplaced)
-    (property "Reference" "J4" (at 202.565 106.68 0)
-      (effects (font (size 1.27 1.27)))
-    )
-    (property "Value" "PN532 connector" (at 202.565 109.22 0)
-      (effects (font (size 1.27 1.27)))
-    )
-    (property "Footprint" "Connector_PinHeader_1.00mm:PinHeader_1x04_P1.00mm_Vertical" (at 201.93 114.3 0)
-      (effects (font (size 1.27 1.27)) hide)
-    )
-    (property "Datasheet" "~" (at 201.93 114.3 0)
-      (effects (font (size 1.27 1.27)) hide)
-    )
-    (pin "3")
-    (pin "1")
-    (pin "2")
-    (pin "4")
-    (instances
-      (project "projekt1"
-        (path "/5c680b0f-7f46-4261-a30f-11ae0254e690"
-          (reference "J4") (unit 1)
-        )
-      )

Commit message: rc522
Parts:
- removed P1: RFID-RC522-MODULE, RF_Module:ESP-07, symbol rfid-rc522-module:RFID-RC522-MODULE
- added RFID1: RC522, symbol My_Library:RC522
Connections:
- net GND: now also RFID1.6 (GND)
- net I2C1_SCL: now also RFID1.2 (SCK)
- net I2C1_SDA: now also RFID1.1 (SDA)
- net VDD: now also RFID1.8 (3,3V)

Commit message: rc522 saved pcb
Parts:
- RFID1: footprint (none) -> My_Footprints_Library:RC522_I2C_B30x20mm
Changed lines of the file:
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@@
       (effects (font (size 1.524 1.524)))
     )
-    (property "Footprint" "" (at 147.32 107.95 0)
+    (property "Footprint" "My_Footprints_Library:RC522_I2C_B30x20mm" (at 147.32 107.95 0)
       (effects (font (size 1.524 1.524)) hide)
     )
