File: projekt1.kicad_sch (KiCad schematic)
At the start: 71 parts, among them IC1 TPS563300DRLR, J1 V1, J2 V1, K1 1461103-1, K2 SANYOU_SRD_Form_B, Q1 MMBT3904, Q2 MMBT3904, SW1 SW_Push, SW10 SW_Push, SW11 SW_Push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

Commit message: cleanup
Other:
- note added: "Keyboard"
- note added: "RFID Module"
- note removed: "Klawiatura"
- moved on the sheet: C10, C12, C14, C16, C8, D1, D10, D11, D12, D2, D3, D4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

Commit message: lecturer remarks fixes
Parts:
- added J3: V1, TerminalBlock_TE-Connectivity:TerminalBlock_TE_282834-2_1x02_P2.54mm_Horizontal, symbol Connector:Conn_01x02_Pin
Connections:
- net +24V: now also J3.2 (Pin_2)
- net GND: now also J3.1 (Pin_1)
Other:
- moved on the sheet: J1, J2
Changed lines of the file:
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@@
     (stroke (width 0) (type default))
   )
+  (wire (pts (xy 117.475 109.22) (xy 117.475 109.855))
+    (stroke (width 0) (type default))
+  )
   (wire (pts (xy 267.335 137.16) (xy 269.875 137.16))
     (stroke (width 0) (type default))
@@
     (stroke (width 0) (type default))
   )
+  (wire (pts (xy 118.745 109.22) (xy 117.475 109.22))
+    (stroke (width 0) (type default))
+  )
   (polyline (pts (xy 176.53 163.83) (xy 176.53 163.83))
     (stroke (width 0) (type dash))
@@
     (effects (font (size 1.27 1.27)) (justify right bottom))
   )
-  (label "COM_V2" (at 118.11 97.79 180) (fields_autoplaced)
+  (label "COM_V2" (at 118.745 92.71 180) (fields_autoplaced)
     (effects (font (size 1.27 1.27)) (justify right bottom))
   )
@@
     (effects (font (size 1.27 1.27)) (justify left bottom))
   )
+  (label "+24V" (at 118.745 106.68 180) (fields_autoplaced)
+    (effects (font (size 1.27 1.27)) (justify right bottom))
+  )
   (label "V1_Open" (at 198.12 34.29 180) (fields_autoplaced)
     (effects (font (size 1.27 1.27)) (justify right bottom))
@@
     (effects (font (size 1.27 1.27)) (justify left bottom))
   )
-  (label "Relay2_NC" (at 118.11 95.25 180) (fields_autoplaced)
+  (label "Relay2_NC" (at 118.745 90.17 180) (fields_autoplaced)
     (effects (font (size 1.27 1.27)) (justify right bottom))
   )
-  (label "+24V" (at 118.11 110.49 180) (fields_autoplaced)
+  (label "+24V" (at 118.745 100.965 180) (fields_autoplaced)
     (effects (font (size 1.27 1.27)) (justify right bottom))
   )
@@
     (effects (font (size 1.27 1.27)) (justify right bottom))
   )
-  (label "Relay1_NO" (at 118.11 107.95 180) (fields_autoplaced)
+  (label "Relay1_NO" (at 118.745 98.425 180) (fields_autoplaced)
     (effects (font (size 1.27 1.27)) (justify right bottom))
   )
@@
     )
   )
-  (symbol (lib_id "Connector:Conn_01x02_Pin") (at 123.19 110.49 180) (unit 1)
+  (symbol (lib_id "Connector:Conn_01x02_Pin") (at 123.825 100.965 180) (unit 1)
     (in_bom yes) (on_board yes) (dnp no)
-    (property "Reference" "J2" (at 124.46 107.95 0)
+    (property "Reference" "J2" (at 125.095 98.425 0)
       (effects (font (size 1.27 1.27)) (justify right))
     )
-    (property "Value" "V1" (at 124.46 110.49 0)
+    (property "Value" "V1" (at 125.095 100.965 0)
       (effects (font (size 1.27 1.27)) (justify right))
     )
-    (property "Footprint" "TerminalBlock_TE-Connectivity:TerminalBlock_TE_282834-2_1x02_P2.54mm_Horizontal" (at 123.19 110.49 0)
+    (property "Footprint" "TerminalBlock_TE-Connectivity:TerminalBlock_TE_282834-2_1x02_P2.54mm_Horizontal" (at 123.825 100.965 0)
       (effects (font (size 1.27 1.27)) hide)
     )
-    (property "Datasheet" "~" (at 123.19 110.49 0)
+    (property "Datasheet" "~" (at 123.825 100.965 0)
       (effects (font (size 1.27 1.27)) hide)
     )
@@
     )
   )
-  (symbol (lib_id "Connector:Conn_01x02_Pin") (at 123.19 97.79 180) (unit 1)
+  (symbol (lib_id "Connector:Conn_01x02_Pin") (at 123.825 92.71 180) (unit 1)
     (in_bom yes) (on_board yes) (dnp no)
-    (property "Reference" "J1" (at 124.46 95.25 0)
+    (property "Reference" "J1" (at 125.095 90.17 0)
       (effects (font (size 1.27 1.27)) (justify right))
     )
-    (property "Value" "V1" (at 124.46 97.79 0)
+    (property "Value" "V1" (at 125.095 92.71 0)
       (effects (font (size 1.27 1.27)) (justify right))
     )
-    (property "Footprint" "TerminalBlock:TerminalBlock_Altech_AK300-2_P5.00mm" (at 123.19 97.79 0)
+    (property "Footprint" "TerminalBlock:TerminalBlock_Altech_AK300-2_P5.00mm" (at 123.825 92.71 0)
       (effects (font (size 1.27 1.27)) hide)
     )
-    (property "Datasheet" "~" (at 123.19 97.79 0)
+    (property "Datasheet" "~" (at 123.825 92.71 0)
       (effects (font (size 1.27 1.27)) hide)
     )
@@
     )
   )
+  (symbol (lib_id "Connector:Conn_01x02_Pin") (at 123.825 109.22 180) (unit 1)
+    (in_bom yes) (on_board yes) (dnp no)
+    (property "Reference" "J3" (at 125.095 106.68 0)
+      (effects (font (size 1.27 1.27)) (justify right))
+    )
+    (property "Value" "V1" (at 125.095 109.22 0)
+      (effects (font (size 1.27 1.27)) (justify right))
+    )
+    (property "Footprint" "TerminalBlock_TE-Connectivity:TerminalBlock_TE_282834-2_1x02_P2.54mm_Horizontal" (at 123.825 109.22 0)
+      (effects (font (size 1.27 1.27)) hide)
+    )
+    (property "Datasheet" "~" (at 123.825 109.22 0)
+      (effects (font (size 1.27 1.27)) hide)
+    )
+    (pin "1")
+    (pin "2")
+    (instances
+      (project "projekt1"
+        (path "/5c680b0f-7f46-4261-a30f-11ae0254e690"
+          (reference "J3") (unit 1)
+        )
+      )
+    )
+  )
   (symbol (lib_id "power:+24V") (at 265.43 34.29 270) (unit 1)
     (in_bom yes) (on_board yes) (dnp no) (fields_autoplaced)
@@
         )
       )
+    )
+  )
+  (symbol (lib_id "power:GND") (at 117.475 109.855 0) (unit 1)
+    (in_bom yes) (on_board yes) (dnp no) (fields_autoplaced)
+    (property "Reference" "#PWR019" (at 117.475 116.205 0)
+      (effects (font (size 1.27 1.27)) hide)
+    )
+    (property "Value" "GND" (at 117.475 114.935 0)
+      (effects (font (size 1.27 1.27)))
+    )
+    (property "Footprint" "" (at 117.475 109.855 0)
+      (effects (font (size 1.27 1.27)) hide)
+    )
+    (property "Datasheet" "" (at 117.475 109.855 0)
+      (effects (font (size 1.27 1.27)) hide)
+    )
+    (pin "1")
+    (instances
+      (project "projekt1"
+        (path "/5c680b0f-7f46-4261-a30f-11ae0254e690"
+          (reference "#PWR019") (unit 1)
+        )
+      )
+      (project "KontrolaDostepu"
+        (path "/e73816df-ff4c-47c2-ad95-54701b1a57bc"
+          (reference "#PWR?") (unit 1)
+        )
+      )
