File: projekt1.kicad_pcb (KiCad board)
At the start: 2 copper layers, 184.6 x 41.6 mm, 71 parts, among them IC1 TPS563300DRLR, J1 V1, J2 V1, K1 1461103-1, K2 SANYOU_SRD_Form_B, Q1 MMBT3904, Q2 MMBT3904, SW1 SW_Push, SW10 SW_Push, SW11 SW_Push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

Commit message: cleanup
Parts:
- moved SW3 14.2 mm to (117.5, 108.4)
- moved SW1 14.2 mm to (117.5, 88.3)
- moved SW2 14.2 mm to (117.5, 98.3)
- moved C1 14.2 mm to (158.8, 89.8)
- moved C11 14.2 mm to (164.4, 94.6)
- moved C12 14.2 mm to (106.2, 96.2)
- moved C13 14.2 mm to (177.9, 106.3)
- moved C16 14.2 mm to (99.5, 90.3)
- moved C17 14.2 mm to (176.4, 106.3)
- moved C2 14.2 mm to (169.0, 86.6)
- moved C3 14.2 mm to (169.0, 84.9)
- moved C4 14.2 mm to (169.0, 83.1)
- moved C6 14.2 mm to (157.1, 95.9)
- moved C7 14.2 mm to (169.0, 81.6)
- moved C9 14.2 mm to (166.2, 94.6)
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Routing:
- net /ROW0: track 74.4 -> 70.2 mm
- net /COL2: track 86.9 -> 83.7 mm
- net /COL1: track 101.1 -> 98.1 mm
- net /COL0: track 150.7 -> 147.7 mm
- net /V2_Close: track 80.3 -> 78.4 mm
- net /V1_Open: track 73.6 -> 71.7 mm
- net /ROW3: track 85.5 -> 83.6 mm
- net /I2C1_SDA: track 20.1 -> 18.7 mm

Commit message: spilled gnd layer
Routing:
- net GND: track 0.00 -> 52.1 mm, vias 0 -> 20
- added copper zone on B.Cu, net GND

Commit message: lecturer remarks fixes
Parts:
- added J3: V1, TerminalBlock_TE-Connectivity:TerminalBlock_TE_282834-2_1x02_P2.54mm_Horizontal, F.Cu at (63.4, 116.9)
- moved J2 5.67 mm to (63.4, 107.5)
- moved K1 2.34 mm to (90.6, 108.0)
Routing:
- net /COM_V2: track 18.6 -> 0.00 mm
- net /Relay2_NC: track 10.1 -> 0.00 mm
- net +24V: track 206.0 -> 215.5 mm
- net /Relay1_NO: track 7.09 -> 14.0 mm
- net GND: track 52.1 -> 54.5 mm, vias 20 -> 21
- net Net-(D14-A): track 7.09 -> 5.58 mm
- added copper zone on F.Cu, net /COM_V2
- added copper zone on F.Cu, net /Relay2_NC
Other:
- board text added: "Kontrola dostępu v1.0 Kacper Nowaczyk 150616 Robert Dobrowolski 147572"
